Commit message: ENH: costmap done

File: src/robot_model/urdf/fishbot_gazebo.urdf (robot description, URDF)
Before this commit: robot fishbot, 8 links, 7 joints
Joints:
- joint left_wheel_joint: origin xyz=-0.02 0.10 -0.06 -> xyz=0 0.10 -0.06
- joint right_wheel_joint: origin xyz=-0.02 -0.10 -0.06 -> xyz=0 -0.10 -0.06

Commit message: ENH: more code

File: src/robot_model/urdf/fishbot_gazebo.urdf (robot description, URDF)
Before this commit: robot fishbot, 8 links, 7 joints
Joints:
- joint imu_joint: origin xyz=0 0 0.02 -> xyz=0 0 0
