Commit message: fix urdf && build map

File: src/robot_model/urdf/fishbot_gazebo.urdf (robot description, URDF)
Before this commit: robot fishbot, 8 links, 7 joints
Links:
- removed link caster_link
- removed link caster_link1
- added link rear_caster_swivel_link, mass 0.05; collision box size=0.018 0.018 0.012; visual box size=0.018 0.018 0.012
- added link rear_caster_wheel_link, mass 0.13; collision cylinder length=0.012 radius=0.018; visual cylinder length=0.012 radius=0.018
- link base_link: mass 0.2 -> 6.0; geometry collision cylinder length=0.08 radius=0.12; visual cylinder length=0.08 radius=0.12
- link imu_link: mass 0.1 -> 0.03
- link laser_link: mass 0.1 -> 0.05
- link left_wheel_link: mass 0.2 -> 0.35
- link right_wheel_link: mass 0.2 -> 0.35
Joints:
- removed joint caster_joint
- removed joint caster_joint1
- added joint rear_caster_swivel_joint: type continuous, parent base_link, child rear_caster_swivel_link, origin xyz=-0.105 0.0 -0.002, axis 0 0 1
- added joint rear_caster_wheel_joint: type continuous, parent rear_caster_swivel_link, child rear_caster_wheel_link, origin xyz=-0.015 0.0 -0.027, axis 0 1 0
- joint base_joint: origin xyz=0.0 0.0 0.076 rpy=0 0 0 -> xyz=0.0 0.0 0.047 rpy=0 0 0
- joint laser_joint: origin xyz=0 0 0.075 -> xyz=0 0 0.04
- joint left_wheel_joint: origin xyz=0 0.10 -0.06 -> xyz=0.0 0.10 -0.015
- joint right_wheel_joint: origin xyz=0 -0.10 -0.06 -> xyz=0.0 -0.10 -0.015

Commit message: add camera

File: src/robot_model/urdf/fishbot_gazebo.urdf (robot description, URDF)
Before this commit: robot fishbot, 8 links, 7 joints
Links:
- added link camera_link, mass 0.08; collision box size=0.04 0.08 0.04; visual box size=0.04 0.08 0.04
Joints:
- added joint camera_joint: type fixed, parent base_link, child camera_link, origin xyz=0.145 0 0.08 rpy=0 0 0

Commit message: fix camera

File: src/robot_model/urdf/fishbot_gazebo.urdf (robot description, URDF)
Before this commit: robot fishbot, 9 links, 8 joints
Joints:
- joint camera_joint: origin xyz=0.145 0 0.08 rpy=0 0 0 -> xyz=0.10 0 0.08 rpy=0 0 0
